File: circuit-board/chcp_schematic.brd (EAGLE design)
At the start: 91.4 x 66 mm, 16 parts, among them IC1 ATMEGA328-20P, IC2 24MAC402, J1 FTDI, J2 LCD1, J3 LCD2, Q1 16 MHz

Commit message: Added 3mm Green Power LED
Parts:
- added LED1: GREEN, led:LED3MM
- added R2: 56R, rcl:0204/7
- moved S1 2.84 mm to (83.8, 59.7), turned to 180 degrees
- moved J2 2.54 mm to (45.7, 52.1)
Connections:
- new net N$8: LED1.A, R2.1
- net +3V3: now also R2.2
- net GND: now also LED1.K
Routing:
- net N$8: track 0.00 -> 7.62 mm
- net +3V3: track 255.9 -> 261.0 mm
- net MOSI: track 127.6 -> 132.7 mm
- net LCD-SS: track 86.4 -> 91.4 mm
- net LCD-RESET: track 101.6 -> 106.7 mm
- net LCD-DC: track 81.3 -> 86.4 mm
- net SCLK: track 117.5 -> 122.6 mm
- net LCD-LIGHT: track 35.6 -> 38.1 mm
- net GND: track 35.6 -> 38.1 mm
